File: pcb/main/pcb.kicad_pcb (KiCad board)
At the start: 4 copper layers, 35.9 x 65 mm, 45 parts, among them J1 Conn_01x04, J2 USB_B_Micro, J6 Barrel_Jack_MountingPin, Q1 Q_NMOS_GDS, Q3 Q_NMOS_GDS, U2 ESP32-C3-WROOM-02, U5 IX4427N, U6 LMR54406DBVR

Commit message: pcb: update part # for esp32
Parts:
- U2: value ESP32-C3-WROOM-02 -> ESP32-C3-WROOM-02-N4
Changed lines of the file:
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@@
 			)
 		)
-		(property "Value" "ESP32-C3-WROOM-02"
+		(property "Value" "ESP32-C3-WROOM-02-N4"
 			(at 0 8 0)
 			(layer "F.Fab")
@@
 			(at 0 0 180)
 			(unlocked yes)
+			(layer "F.Fab")
+			(hide yes)
+			(effects
+				(font
+					(size 1 1)
+					(thickness 0.15)
+				)
+			)
+		)
+		(property "LCSC Part #" "C2934560"
+			(at 0 0 180)
+			(unlocked yes)
